Commit message: fixed urdf errors

File: mono_observer_description/urdf/camera_sensor.xacro (robot description, xacro)
@@ -42,5 +42,5 @@
                     </ros>
                     <camera_name>camera</camera_name>
-                    <frame_name>camera_frame</frame_name>
+                    <frame_name>camera_link</frame_name>
                     <hack_baseline>0.2</hack_baseline>
                 </plugin>

File: mono_observer_description/urdf/mono_observer_urdf.xacro (robot description, xacro)
@@ -3,5 +3,5 @@
     <link name="base_link">
         <visual>
-            <origin xyz="0 0 0" rpy="0 0 0"/>
+            <origin xyz="0 0 0.01" rpy="0 0 0"/>
             <geometry>
                 <box size="0.1 0.1 0.02"/>
@@ -12,5 +12,5 @@
         </visual>
         <collision>
-            <origin xyz="0 0 0" rpy="0 0 0"/>
+            <origin xyz="0 0 0.01" rpy="0 0 0"/>
             <geometry>
                 <box size="0.1 0.1 0.02"/>
@@ -20,7 +20,7 @@
     <link name="link_1">
         <visual>
-            <origin xyz="0 0 0" rpy="0 0 0"/>
+            <origin xyz="0 0 0.05" rpy="0 0 0"/>
             <geometry>
-                <box size="0.01 0.01 0.1"/>
+                <box size="0.03 0.03 0.1"/>
             </geometry>
             <material name="">
@@ -29,5 +29,39 @@
         </visual>
         <collision>
-            <origin xyz="0 0 0" rpy="0 0 0"/>
+            <origin xyz="0 0 0.05" rpy="0 0 0"/>
+            <geometry>
+                <box size="0.01 0.01 0.1"/>
+            </geometry>
+        </collision>
+    </link>
+    <link name="link_2">
+        <visual>
+            <origin xyz="0 0 0.05" rpy="0 0 0"/>
+            <geometry>
+                <box size="0.03 0.03 0.1"/>
+            </geometry>
+            <material name="">
+                <color rgba="0 1 0 1"/>
+            </material>
+        </visual>
+        <collision>
+            <origin xyz="0 0 0.05" rpy="0 0 0"/>
+            <geometry>
+                <box size="0.01 0.01 0.1"/>
+            </geometry>
+        </collision>
+    </link>
+    <link name="link_3">
+        <visual>
+            <origin xyz="0 0 0.05" rpy="0 0 0"/>
+            <geometry>
+                <box size="0.03 0.03 0.1"/>
+            </geometry>
+            <material name="">
+                <color rgba="0 0 1 1"/>
+            </material>
+        </visual>
+        <collision>
+            <origin xyz="0 0 0.05" rpy="0 0 0"/>
             <geometry>
                 <box size="0.01 0.01 0.1"/>
@@ -36,9 +70,23 @@
     </link>
     <joint name="base_1_joint" type="revolute">
-        <origin xyz="0 0 0" rpy="0 0 0"/>
+        <origin xyz="0 0 0.02" rpy="0 0 0"/>
         <parent link="base_link"/>
         <child link="link_1"/>
         <axis xyz="0 0 1" rpy="0 0 0"/>
-        <limit lower="-1.57" upper="1.57"/>
+        <limit effort="30" velocity="1.0" lower="-1.5708" upper="1.5708" />
+    </joint>
+    <joint name="1_2_joint" type="revolute">
+        <origin xyz="0 0 0.1" rpy="0 0 0"/>
+        <parent link="link_1"/>
+        <child link="link_2"/>
+        <axis xyz="1 0 0" rpy="0 0 0"/>
+        <limit effort="30" velocity="1.0" lower="-1.5708" upper="1.5708" />
+    </joint>
+    <joint name="2_3_joint" type="revolute">
+        <origin xyz="0 0 0.1" rpy="0 0 0"/>
+        <parent link="link_2"/>
+        <child link="link_3"/>
+        <axis xyz="1 0 0" rpy="0 0 0"/>
+        <limit effort="30" velocity="1.0" lower="-1.5708" upper="1.5708" />
     </joint>
 </robot>
