Commit message: add mjcf, mujoco controller, and config file

File: mono_observer_description/urdf/mono_observer_controller.xacro (robot description, xacro)
@@ -4,4 +4,5 @@
     <xacro:include filename="$(find ${package_name})/urdf/xacro_properties.xacro"/>
     <xacro:include filename="$(find ${package_name})/urdf/mono_observer_urdf.xacro"/>
+    <xacro:include filename="$(find ${package_name})/urdf/trajectory_controller.xacro"/>
     <!--<xacro:include filename="$(find ${package_name})/urdf/camera_sensor.xacro"/>-->
 </robot>

File: mono_observer_description/urdf/mono_observer_urdf.xacro (robot description, xacro)
@@ -7,5 +7,5 @@
                 <mesh filename="${base_mesh}"/>
             </geometry>
-            <material name="">
+            <material name="gray">
                 <color rgba="0.7 0.7 0.7 1"/>
             </material>
@@ -24,5 +24,5 @@
                 <mesh filename="${cintura_mesh}"/>
             </geometry>
-            <material name="">
+            <material name="red">
                 <color rgba="1 0 0 1"/>
             </material>
@@ -41,5 +41,5 @@
                 <mesh filename="${antebrazo_mesh}"/>
             </geometry>
-            <material name="">
+            <material name="green">
                 <color rgba="0 1 0 1"/>
             </material>
@@ -58,5 +58,5 @@
                 <mesh filename="${soporte_camara_mesh}"/>
             </geometry>
-            <material name="">
+            <material name="blue">
                 <color rgba="0 0 1 1"/>
             </material>
