Commit message: fix urdf joint limits

File: mono_observer_description/urdf/mono_observer_urdf.xacro (robot description, xacro)
@@ -81,5 +81,5 @@
         <child link="link_2"/>
         <axis xyz="1 0 0" rpy="0 0 0"/>
-        <limit effort="30" velocity="1.0" lower="-1.5708" upper="1.5708" />
+        <limit effort="30" velocity="1.0" lower="0" upper="3.1416" />
     </joint>
     <joint name="2_3_joint" type="revolute">
@@ -88,5 +88,5 @@
         <child link="link_3"/>
         <axis xyz="1 0 0" rpy="0 0 0"/>
-        <limit effort="30" velocity="1.0" lower="-1.5708" upper="1.5708" />
+        <limit effort="30" velocity="1.0" lower="0" upper="3.1416" />
     </joint>
 </robot>

Commit message: add mesh to urdf

File: mono_observer_description/urdf/mono_observer_urdf.xacro (robot description, xacro)
@@ -5,5 +5,5 @@
             <origin xyz="0 0 0.01" rpy="0 0 0"/>
             <geometry>
-                <box size="0.1 0.1 0.02"/>
+                <mesh filename="${base_mesh}"/>
             </geometry>
             <material name="">

Commit message: add fixed meshes for cintura and base

File: mono_observer_description/urdf/mono_observer_urdf.xacro (robot description, xacro)
@@ -3,5 +3,5 @@
     <link name="base_link">
         <visual>
-            <origin xyz="0 0 0.01" rpy="0 0 0"/>
+            <origin xyz="0 0 0" rpy="0 0 0"/>
             <geometry>
                 <mesh filename="${base_mesh}"/>
@@ -20,7 +20,7 @@
     <link name="link_1">
         <visual>
-            <origin xyz="0 0 0.05" rpy="0 0 0"/>
+            <origin xyz="0 0 -0.02" rpy="0 0 0"/>
             <geometry>
-                <box size="0.03 0.03 0.1"/>
+                <mesh filename="${cintura_mesh}"/>
             </geometry>
             <material name="">

File: mono_observer_description/urdf/xacro_properties.xacro (robot description, xacro)
@@ -1,4 +1,5 @@
 <?xml version="1.0" encoding="utf-8"?>
 <robot xmlns:xacro="http://ros.org/wiki/xacro" >
-    <xacro:property name="base_mesh" value="package://mono_observer_description/meshes/stl_V1/Base.stl"/>
+    <xacro:property name="base_mesh" value="package://mono_observer_description/meshes/Base.stl"/>
+    <xacro:property name="cintura_mesh" value="package://mono_observer_description/meshes/Cintura.stl"/>
 </robot>

Commit message: add antebrazo

File: mono_observer_description/urdf/mono_observer_urdf.xacro (robot description, xacro)
@@ -37,7 +37,7 @@
     <link name="link_2">
         <visual>
-            <origin xyz="0 0 0.05" rpy="0 0 0"/>
+            <origin xyz="0 0 -0.08" rpy="0 0 0"/>
             <geometry>
-                <box size="0.03 0.03 0.1"/>
+                <mesh filename="${antebrazo_mesh}"/>
             </geometry>
             <material name="">

File: mono_observer_description/urdf/xacro_properties.xacro (robot description, xacro)
@@ -3,3 +3,4 @@
     <xacro:property name="base_mesh" value="package://mono_observer_description/meshes/Base.stl"/>
     <xacro:property name="cintura_mesh" value="package://mono_observer_description/meshes/Cintura.stl"/>
+    <xacro:property name="antebrazo_mesh" value="package://mono_observer_description/meshes/Antebrazo.stl"/>
 </robot>

Commit message: add last mesh, fix antebrazo mesh

File: mono_observer_description/urdf/mono_observer_urdf.xacro (robot description, xacro)
@@ -20,5 +20,5 @@
     <link name="link_1">
         <visual>
-            <origin xyz="0 0 -0.02" rpy="0 0 0"/>
+            <origin xyz="0 0 -0.05" rpy="0 0 0"/>
             <geometry>
                 <mesh filename="${cintura_mesh}"/>
@@ -54,7 +54,7 @@
     <link name="link_3">
         <visual>
-            <origin xyz="0 0 0.05" rpy="0 0 0"/>
+            <origin xyz="0 0 -0.15" rpy="0 0 0"/>
             <geometry>
-                <box size="0.03 0.03 0.1"/>
+                <mesh filename="${soporte_camara_mesh}"/>
             </geometry>
             <material name="">
@@ -70,5 +70,5 @@
     </link>
     <joint name="base_1_joint" type="revolute">
-        <origin xyz="0 0 0.02" rpy="0 0 0"/>
+        <origin xyz="0 0 0.05" rpy="0 0 0"/>
         <parent link="base_link"/>
         <child link="link_1"/>
@@ -77,15 +77,15 @@
     </joint>
     <joint name="1_2_joint" type="revolute">
-        <origin xyz="0 0 0.1" rpy="0 0 0"/>
+        <origin xyz="0 0 0.03" rpy="0 0 0"/>
         <parent link="link_1"/>
         <child link="link_2"/>
-        <axis xyz="1 0 0" rpy="0 0 0"/>
+        <axis xyz="0 1 0" rpy="0 0 0"/>
         <limit effort="30" velocity="1.0" lower="0" upper="3.1416" />
     </joint>
     <joint name="2_3_joint" type="revolute">
-        <origin xyz="0 0 0.1" rpy="0 0 0"/>
+        <origin xyz="0 0 0.071" rpy="0 0 0"/>
         <parent link="link_2"/>
         <child link="link_3"/>
-        <axis xyz="1 0 0" rpy="0 0 0"/>
+        <axis xyz="0 1 0" rpy="0 0 0"/>
         <limit effort="30" velocity="1.0" lower="0" upper="3.1416" />
     </joint>

File: mono_observer_description/urdf/xacro_properties.xacro (robot description, xacro)
@@ -4,3 +4,4 @@
     <xacro:property name="cintura_mesh" value="package://mono_observer_description/meshes/Cintura.stl"/>
     <xacro:property name="antebrazo_mesh" value="package://mono_observer_description/meshes/Antebrazo.stl"/>
+    <xacro:property name="soporte_camara_mesh" value="package://mono_observer_description/meshes/Camara.stl"/>
 </robot>

Commit message: add litle introduction and fix servo range

File: mono_observer_description/urdf/mono_observer_urdf.xacro (robot description, xacro)
@@ -81,5 +81,5 @@
         <child link="link_2"/>
         <axis xyz="0 1 0" rpy="0 0 0"/>
-        <limit effort="30" velocity="1.0" lower="0" upper="3.1416" />
+        <limit effort="30" velocity="1.0" lower="-1.5708" upper="1.5708" />
     </joint>
     <joint name="2_3_joint" type="revolute">
@@ -88,5 +88,5 @@
         <child link="link_3"/>
         <axis xyz="0 1 0" rpy="0 0 0"/>
-        <limit effort="30" velocity="1.0" lower="0" upper="3.1416" />
+        <limit effort="30" velocity="1.0" lower="-1.5708" upper="1.5708" />
     </joint>
 </robot>

Commit message: fix urdf colision and rviz viewpoint

File: mono_observer_description/urdf/mono_observer_urdf.xacro (robot description, xacro)
@@ -12,7 +12,7 @@
         </visual>
         <collision>
-            <origin xyz="0 0 0.01" rpy="0 0 0"/>
+            <origin xyz="-0.0075 0 0.02" rpy="0 0 0"/>
             <geometry>
-                <box size="0.1 0.1 0.02"/>
+                <box size="0.06 0.03 0.04"/>
             </geometry>
         </collision>
@@ -77,9 +77,9 @@
     </joint>
     <joint name="1_2_joint" type="revolute">
-        <origin xyz="0 0 0.03" rpy="0 0 0"/>
+        <origin xyz="0 0 0.03" rpy="0 1.5708 0"/>
         <parent link="link_1"/>
         <child link="link_2"/>
         <axis xyz="0 1 0" rpy="0 0 0"/>
-        <limit effort="30" velocity="1.0" lower="-1.5708" upper="1.5708" />
+        <limit effort="30" velocity="1.0" lower="-3.1415" upper="0" />
     </joint>
     <joint name="2_3_joint" type="revolute">
