Commit message: add gazebo testing files

File: mono_observer_description/urdf/mono_observer_controller_gz.xacro (robot description, xacro)
@@ -3,7 +3,6 @@
     <xacro:property name="package_name" value="mono_observer_description" />
     <xacro:include filename="$(find ${package_name})/urdf/xacro_properties.xacro"/>
-    <xacro:include filename="$(find ${package_name})/urdf/mujoco_config.xacro"/>
     <xacro:include filename="$(find ${package_name})/urdf/mono_observer_urdf.xacro"/>
-    <xacro:include filename="$(find ${package_name})/urdf/trajectory_controller.xacro"/>
+    <xacro:include filename="$(find ${package_name})/urdf/trajectory_controller_gz.xacro"/>
     <!--<xacro:include filename="$(find ${package_name})/urdf/camera_sensor.xacro"/>-->
 </robot>

File: mono_observer_description/urdf/mono_observer_urdf.xacro (robot description, xacro)
@@ -2,4 +2,9 @@
 <robot xmlns:xacro="http://ros.org/wiki/xacro">
     <link name="base_link">
+        <inertial>
+            <origin xyz="0.0 0.0 0.0" rpy="0 0 0" />
+            <mass value="0.02" />
+            <inertia ixx="1" ixy="0" ixz="0" iyy="1" iyz="0" izz="1" />
+        </inertial>
         <visual>
             <origin xyz="0 0 0" rpy="0 0 0"/>
@@ -19,4 +24,9 @@
     </link>
     <link name="link_1">
+        <inertial>
+            <origin xyz="0.0 0.0 0.0" rpy="0 0 0" />
+            <mass value="0.02" />
+            <inertia ixx="1" ixy="0" ixz="0" iyy="1" iyz="0" izz="1" />
+        </inertial>
         <visual>
             <origin xyz="0 0 -0.05" rpy="0 0 0"/>
@@ -29,11 +39,16 @@
         </visual>
         <collision>
-            <origin xyz="0 0 0.05" rpy="0 0 0"/>
+            <origin xyz="0 0 0" rpy="0 0 0"/>
             <geometry>
-                <box size="0.01 0.01 0.1"/>
+                <box size="0.03 0.03 0.01"/>
             </geometry>
         </collision>
     </link>
     <link name="link_2">
+        <inertial>
+            <origin xyz="0.0 0.0 0.0" rpy="0 0 0" />
+            <mass value="0.02" />
+            <inertia ixx="1" ixy="0" ixz="0" iyy="1" iyz="0" izz="1" />
+        </inertial>
         <visual>
             <origin xyz="0 0 -0.08" rpy="0 0 0"/>
@@ -46,11 +61,16 @@
         </visual>
         <collision>
-            <origin xyz="0 0 0.05" rpy="0 0 0"/>
+            <origin xyz="0 0 0.01" rpy="0 0 0"/>
             <geometry>
-                <box size="0.01 0.01 0.1"/>
+                <box size="0.04 0.03 0.05"/>
             </geometry>
         </collision>
     </link>
     <link name="link_3">
+        <inertial>
+            <origin xyz="0.0 0.0 0.0" rpy="0 0 0" />
+            <mass value="0.02" />
+            <inertia ixx="1" ixy="0" ixz="0" iyy="1" iyz="0" izz="1" />
+        </inertial>
         <visual>
             <origin xyz="0 0 -0.15" rpy="0 0 0"/>
@@ -63,7 +83,7 @@
         </visual>
         <collision>
-            <origin xyz="0 0 0.05" rpy="0 0 0"/>
+            <origin xyz="0 0 0.0075" rpy="0 0 0"/>
             <geometry>
-                <box size="0.01 0.01 0.1"/>
+                <box size="0.04 0.03 0.05"/>
             </geometry>
         </collision>
@@ -74,5 +94,5 @@
         <child link="link_1"/>
         <axis xyz="0 0 1" rpy="0 0 0"/>
-        <limit effort="30" velocity="1.0" lower="-1.5708" upper="1.5708" />
+        <limit effort="30" velocity="1.0" lower="-3.1415" upper="0" />
     </joint>
     <joint name="1_2_joint" type="revolute">
@@ -84,9 +104,9 @@
     </joint>
     <joint name="2_3_joint" type="revolute">
-        <origin xyz="0 0 0.071" rpy="0 0 0"/>
+        <origin xyz="0 0 0.071" rpy="0 1.5708 0"/>
         <parent link="link_2"/>
         <child link="link_3"/>
         <axis xyz="0 1 0" rpy="0 0 0"/>
-        <limit effort="30" velocity="1.0" lower="-1.5708" upper="1.5708" />
+        <limit effort="30" velocity="1.0" lower="-3.1415" upper="0" />
     </joint>
 </robot>
