Commit message: add mujoco and gazebo(test) launch files

File: mono_observer_description/mujoco_models/full_xacro.urdf (robot description, URDF)
Before this commit: robot mono_observer, 4 links, 3 joints
Links:
- link base_link: mass None -> 0.02; geometry collision box size=0.06 0.03 0.04; visual mesh filename=package://mono_observer_description/meshes/Base.stl
- link link_1: mass None -> 0.02; geometry collision box size=0.03 0.03 0.01; visual mesh filename=package://mono_observer_description/meshes/Cintura.stl
- link link_2: mass None -> 0.02; geometry collision box size=0.04 0.03 0.05; visual mesh filename=package://mono_observer_description/meshes/Antebrazo.stl
- link link_3: mass None -> 0.02; geometry collision box size=0.04 0.03 0.05; visual mesh filename=package://mono_observer_description/meshes/Camara.stl
Joints:
- joint 1_2_joint: limit lower=-1.5708 upper=1.5708 effort=30 velocity=1.0 -> lower=-3.1415 upper=0 effort=30 velocity=1.0; origin xyz=0 0 0.03 rpy=0 0 0 -> xyz=0 0 0.03 rpy=0 1.5708 0
- joint 2_3_joint: limit lower=-1.5708 upper=1.5708 effort=30 velocity=1.0 -> lower=-3.1415 upper=0 effort=30 velocity=1.0; origin xyz=0 0 0.071 rpy=0 0 0 -> xyz=0 0 0.071 rpy=0 1.5708 0
- joint base_1_joint: limit lower=-1.5708 upper=1.5708 effort=30 velocity=1.0 -> lower=-3.1415 upper=0 effort=30 velocity=1.0

Commit message: fixed range in model

File: mono_observer_description/mujoco_models/full_xacro.urdf (robot description, URDF)
Before this commit: robot mono_observer, 4 links, 3 joints
Joints:
- joint 1_2_joint: limit lower=-3.1415 upper=0 effort=30 velocity=1.0 -> lower=-1.5707 upper=1.5707 effort=30 velocity=1.0; origin xyz=0 0 0.03 rpy=0 1.5708 0 -> xyz=0 0 0.03 rpy=0 0 0
- joint 2_3_joint: limit lower=-3.1415 upper=0 effort=30 velocity=1.0 -> lower=-1.5707 upper=1.5707 effort=30 velocity=1.0; origin xyz=0 0 0.071 rpy=0 1.5708 0 -> xyz=0 0 0.071 rpy=0 0 0

File: mono_observer_description/urdf/mono_observer_urdf.xacro (robot description, xacro)
@@ -97,16 +97,16 @@
     </joint>
     <joint name="1_2_joint" type="revolute">
-        <origin xyz="0 0 0.03" rpy="0 1.5708 0"/>
+        <origin xyz="0 0 0.03" rpy="0 0 0"/>
         <parent link="link_1"/>
         <child link="link_2"/>
         <axis xyz="0 1 0" rpy="0 0 0"/>
-        <limit effort="30" velocity="1.0" lower="-3.1415" upper="0" />
+        <limit effort="30" velocity="1.0" lower="-1.5707" upper="1.5707" />
     </joint>
     <joint name="2_3_joint" type="revolute">
-        <origin xyz="0 0 0.071" rpy="0 1.5708 0"/>
+        <origin xyz="0 0 0.071" rpy="0 0 0"/>
         <parent link="link_2"/>
         <child link="link_3"/>
         <axis xyz="0 1 0" rpy="0 0 0"/>
-        <limit effort="30" velocity="1.0" lower="-3.1415" upper="0" />
+        <limit effort="30" velocity="1.0" lower="-1.5707" upper="1.5707" />
     </joint>
 </robot>

Commit message: add Angle testing and changed urdf

File: mono_observer_description/mujoco_models/full_xacro.urdf (robot description, URDF)
Before this commit: robot mono_observer, 4 links, 3 joints
Joints:
- joint base_1_joint: axis 0 0 1 -> 0 0 -1

File: mono_observer_description/urdf/mono_observer_urdf.xacro (robot description, xacro)
@@ -93,5 +93,5 @@
         <parent link="base_link"/>
         <child link="link_1"/>
-        <axis xyz="0 0 1" rpy="0 0 0"/>
+        <axis xyz="0 0 -1" rpy="0 0 0"/>
         <limit effort="30" velocity="1.0" lower="-3.1415" upper="0" />
     </joint>

Commit message: add ToUnity file and interface, fix urdf file

File: mono_observer_description/mujoco_models/full_xacro.urdf (robot description, URDF)
Before this commit: robot mono_observer, 4 links, 3 joints
Joints:
- joint base_1_joint: axis 0 0 -1 -> 0 0 1

File: mono_observer_description/urdf/mono_observer_urdf.xacro (robot description, xacro)
@@ -93,5 +93,5 @@
         <parent link="base_link"/>
         <child link="link_1"/>
-        <axis xyz="0 0 -1" rpy="0 0 0"/>
+        <axis xyz="0 0 1" rpy="0 0 0"/>
         <limit effort="30" velocity="1.0" lower="-3.1415" upper="0" />
     </joint>
